Commit message: update packages

File: bumperbot_ws/src/bumperbot_description/urdf/bumperbot.urdf.xacro (robot description, xacro)
@@ -3,7 +3,10 @@
     <xacro:arg name="is_ignition" default="true" />
     <!-- Add your robot description here -->
-    <xacro:include filename="$(find bumperbot_description)/urdf/bumperbot_gazebo.xacro" />
-    <xacro:include filename="$(find bumperbot_description)/urdf/bumperbot_ros2_control.xacro" />
-    <link name="base_footprint" />
+    <xacro:include
+        filename="$(find bumperbot_description)/urdf/bumperbot_gazebo.xacro" />
+    <xacro:include
+        filename="$(find bumperbot_description)/urdf/bumperbot_ros2_control.xacro" />
+    <link
+        name="base_footprint" />
     <link name="base_link">
         <inertial>
@@ -27,5 +30,6 @@
         </collision>
     </link>
-    <joint name="base_joint" type="fixed">
+    <joint
+        name="base_joint" type="fixed">
         <parent link="base_footprint" />
         <child link="base_link" />
@@ -54,5 +58,6 @@
         </collision>
     </link>
-    <joint name="wheel_right_joint" type="continuous">
+    <joint
+        name="wheel_right_joint" type="continuous">
         <origin xyz="0 -0.0701101849418637 0" rpy="0 0 0" />
         <parent link="base_link" />
@@ -83,5 +88,6 @@
         </collision>
     </link>
-    <joint name="wheel_left_joint" type="continuous">
+    <joint
+        name="wheel_left_joint" type="continuous">
         <origin xyz="0 0.0701101849418642 0" rpy="0 0 0" />
         <parent link="base_link" />
@@ -111,5 +117,6 @@
         </collision>
     </link>
-    <joint name="caster_front_joint" type="fixed">
+    <joint
+        name="caster_front_joint" type="fixed">
         <origin xyz="0.04755 0 -0.0275" rpy="0 0 0" />
         <parent link="base_link" />
@@ -139,5 +146,6 @@
         </collision>
     </link>
-    <joint name="caster_rear_joint" type="fixed">
+    <joint
+        name="caster_rear_joint" type="fixed">
         <origin xyz="-0.04755 0 -0.0275" rpy="0 0 0" />
         <parent link="base_link" />
@@ -145,3 +153,33 @@
         <axis xyz="0 0 0" />
     </joint>
+    <link name="imu_link">
+        <inertial>
+            <origin xyz="-0.00552433659106688 0.000168210391520346 0.000514000497342681" rpy="0 0 0" />
+            <mass value="0.000528415362211671" />
+            <inertia ixx="1.46176048428261E-08" ixy="1.40015117949421E-10" ixz="-1.99633872937403E-12"
+                iyy="8.59662482954888E-09" iyz="7.52375112767959E-12"
+                izz="2.30279421279312E-08" />
+        </inertial>
+        <visual>
+            <origin xyz="0 0 0" rpy="0 0 0" />
+            <geometry>
+                <mesh filename="package://bumperbot_description/meshes/imu_link.STL" />
+            </geometry>
+            <material name="">
+                <color rgba="0.792156862745098 0.819607843137255 0.933333333333333 1" />
+            </material>
+        </visual>
+        <collision>
+            <origin xyz="0 0 0" rpy="0 0 0" />
+            <geometry>
+                <mesh filename="package://bumperbot_description/meshes/imu_link.STL" />
+            </geometry>
+        </collision>
+    </link>
+    <joint name="imu_joint" type="fixed">
+        <origin xyz="0 0 0.0698986241758014" rpy="0 0 0" />
+        <parent link="base_link" />
+        <child link="imu_link" />
+        <axis xyz="0 0 0" />
+    </joint>
 </robot>

File: bumperbot_ws/src/bumperbot_description/urdf/bumperbot_gazebo.xacro (robot description, xacro)
@@ -43,4 +43,7 @@
                <parameters>$(find bumperbot_controller)/config/bumperbot_controllers.yaml</parameters>
             </plugin>
+            <!-- plugin -->
+            <plugin filename="ignition-gazebo-imu-system" name="ignition::gazebo::systems::Imu">
+            </plugin>
         </xacro:if>
         <xacro:unless value="$(arg is_ignition)">
@@ -48,5 +51,48 @@
                 <parameters>$(find bumperbot_controller)/config/bumperbot_controllers.yaml</parameters>
             </plugin>
+            <!-- plugin -->
+            <plugin filename="gz-sim-imu-system" name="gazebo::sim::systems::Imu">
+            </plugin>
         </xacro:unless>
     </gazebo>
+    <gazebo reference="imu_link">
+        <sensor name="imu" type="imu">
+            <always_on>true</always_on>
+            <update_rate>100</update_rate>
+            <gz_frame_is>imu_link</gz_frame_is>
+            <topic>imu</topic>
+            <imu>
+                <angular_velocity>
+                  <x>
+                    <noise type="gaussian">
+                    <mean>0.0</mean>
+                    <stddev>2e-4</stddev>
+                    </noise>
+                   </x>
+                    <y><noise type="gaussian">
+                    <mean>0.0</mean>
+                    <stddev>2e-4</stddev>
+                    </noise>  </y>
+                    <z> <noise type="gaussian">
+                    <mean>0.0</mean>
+                    <stddev>2e-4</stddev>
+                    </noise> </z>
+                </angular_velocity>
+                <linear_acceleration>
+                    <x> <noise type="gaussian">
+                    <mean>0.0</mean>
+                    <stddev>1.7e-2</stddev>
+                    </noise> </x>
+                    <y> <noise type="gaussian">
+                    <mean>0.0</mean>
+                    <stddev>1.7e-2</stddev>
+                    </noise> </y>
+                    <z> <noise type="gaussian">
+                    <mean>0.0</mean>
+                    <stddev>1.7e-2</stddev>
+                    </noise> </z>
+                </linear_acceleration>
+            </imu>
+        </sensor>
+    </gazebo>
 </robot>
